File: circuit/main.kicad_sch (KiCad schematic)
At the start: 17 parts, among them M1 Motor_DC, M2 Motor_DC, U1 VL53L1CXV0FY1, U2 VL53L1CXV0FY1, U3 VL53L1CXV0FY1, U4 L293

Commit message: a
Parts:
- removed C1, C2: 0.1 μF, symbol Device:C
Changed lines of the file:
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@@
   (junction (at 93.98 107.95) (diameter 0) (color 0 0 0 0)
   )
-  (junction (at 223.52 54.61) (diameter 0) (color 0 0 0 0)
-  )
   (junction (at 172.72 147.32) (diameter 0) (color 0 0 0 0)
   )
-  (junction (at 223.52 82.55) (diameter 0) (color 0 0 0 0)
-  )
-  (junction (at 223.52 69.85) (diameter 0) (color 0 0 0 0)
-  )
   (junction (at 58.42 105.41) (diameter 0) (color 0 0 0 0)
   )
@@
   (junction (at 166.37 137.16) (diameter 0) (color 0 0 0 0)
   )
-  (junction (at 223.52 67.31) (diameter 0) (color 0 0 0 0)
-  )
   (junction (at 133.35 127) (diameter 0) (color 0 0 0 0)
   )
@@
     (stroke (width 0) (type default))
   )
-  (wire (pts (xy 241.3 82.55) (xy 223.52 82.55))
-    (stroke (width 0) (type default))
-  )
   (wire (pts (xy 132.08 91.44) (xy 132.08 111.76))
     (stroke (width 0) (type default))
@@
     (stroke (width 0) (type default))
   )
-  (wire (pts (xy 241.3 57.15) (xy 241.3 54.61))
-    (stroke (width 0) (type default))
-  )
   (wire (pts (xy 162.56 93.98) (xy 162.56 105.41))
     (stroke (width 0) (type default))
@@
     (stroke (width 0) (type default))
   )
-  (wire (pts (xy 241.3 67.31) (xy 223.52 67.31))
-    (stroke (width 0) (type default))
-  )
   (wire (pts (xy 127 134.62) (xy 127 137.16))
     (stroke (width 0) (type default))
@@
     (stroke (width 0) (type default))
   )
-  (wire (pts (xy 241.3 69.85) (xy 223.52 69.85))
-    (stroke (width 0) (type default))
-  )
   (wire (pts (xy 147.32 43.18) (xy 198.12 43.18))
     (stroke (width 0) (type default))
@@
     (stroke (width 0) (type default))
   )
-  (wire (pts (xy 241.3 54.61) (xy 223.52 54.61))
-    (stroke (width 0) (type default))
-  )
   (wire (pts (xy 187.96 116.84) (xy 187.96 83.82))
     (stroke (width 0) (type default))
@@
     (stroke (width 0) (type default))
   )
-  (wire (pts (xy 241.3 64.77) (xy 241.3 67.31))
-    (stroke (width 0) (type default))
-  )
   (wire (pts (xy 20.32 105.41) (xy 20.32 66.04))
     (stroke (width 0) (type default))
   )
-  (wire (pts (xy 241.3 80.01) (xy 241.3 82.55))
-    (stroke (width 0) (type default))
-  )
   (wire (pts (xy 60.96 100.33) (xy 60.96 71.12))
     (stroke (width 0) (type default))
@@
   )
   (wire (pts (xy 124.46 102.87) (xy 22.86 102.87))
-    (stroke (width 0) (type default))
-  )
-  (wire (pts (xy 241.3 72.39) (xy 241.3 69.85))
     (stroke (width 0) (type default))
   )
@@
     )
   )
-  (symbol (lib_id "Device:C") (at 241.3 76.2 0) (unit 1)
-    (in_bom yes) (on_board yes) (dnp no) (fields_autoplaced)
-    (property "Reference" "C2" (at 245.11 75.565 0)
-      (effects (font (size 1.27 1.27)) (justify left))
-    )
-    (property "Value" "0.1 μF" (at 245.11 78.105 0)
-      (effects (font (size 1.27 1.27)) (justify left))
-    )
-    (property "Footprint" "" (at 242.2652 80.01 0)
-      (effects (font (size 1.27 1.27)) hide)
-    )
-    (property "Datasheet" "~" (at 241.3 76.2 0)
-      (effects (font (size 1.27 1.27)) hide)
-    )
-    (pin "1")
-    (pin "2")
-    (instances
-      (project "main"
-        (path "/e989136e-5e5c-451b-8d4b-116875cd7499"
-          (reference "C2") (unit 1)
-        )
-      )
-    )
-  )
   (symbol (lib_id "power:GND") (at 152.4 101.6 0) (unit 1)
     (in_bom yes) (on_board yes) (dnp no) (fields_autoplaced)
@@
         )
       )
-    )
-  )
-  (symbol (lib_id "Device:C") (at 241.3 60.96 0) (unit 1)
-    (in_bom yes) (on_board yes) (dnp no) (fields_autoplaced)
-    (property "Reference" "C1" (at 245.11 60.325 0)
-      (effects (font (size 1.27 1.27)) (justify left))
-    )
-    (property "Value" "0.1 μF" (at 245.11 62.865 0)
-      (effects (font (size 1.27 1.27)) (justify left))
-    )
-    (property "Footprint" "" (at 242.2652 64.77 0)
-      (effects (font (size 1.27 1.27)) hide)
-    )
-    (property "Datasheet" "~" (at 241.3 60.96 0)
-      (effects (font (size 1.27 1.27)) hide)
-    )
-    (pin "1")
-    (pin "2")
-    (instances
-      (project "main"
-        (path "/e989136e-5e5c-451b-8d4b-116875cd7499"
-          (reference "C1") (unit 1)
-        )
-      )

Commit message: c
Parts:
- U1, U2, U3: value VL53L1CXV0FY1 -> AE-VL53L
- U4: value L293 -> L293N
- renumbered R5 to R1, R6 to R2, R8 to R3, R9 to R4
Connections:
- net at A1.5 (+5V), D2.2 (A), D3.2 (A)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: now also U1.11 (AVDD), U2.11 (AVDD), U3.11 (AVDD)
